File: Round_LED_Flash.kicad_sch (KiCad schematic)
At the start: 239 parts, among them J1 USB4085-GF-A, J2 BATTERY, J3 BM02B-GHS-TBT(LF)(SN), J4 WARM COB, J5 COOL COB, Q1 AO3400A, Q2 AO3400A, Q20 AO3401A, Q21 AO3401A, Q22 MMBT3904-7-F, Q23 MMBT3904-7-F, Q3 MMBT3904-7-F, Q30 AO3401A, Q31 MMBT3904-7-F, Q32 MMBT3904-7-F, Q33 MMBT3904-7-F, Q34 AO3400A, Q35 MMBT3904-7-F, Q60 AO4407A, Q61 MMBT3904-7-F, Q62 MMBT3904-7-F, Q70 SiR800DP-T1-GE3, SW1 POWER, SW2 SHUTTER, U1 DW01A, U10 ESP32-C3-WROOM-02-N4, U2 TLV76033DBZR, U3 TUSB320LAIRWBR, U30 LTC3225EDDB#TRMPBF, U4 SN74LVC1G04DBVR, U40 LTC6993CS6-1#TRMPBF, U41 LTC6993CS6-1#TRMPBF, U42 TLV3011BIDBVR, U43 TLV3011BIDBVR, U44 SN74LVC1G08DBVR, U45 SN74LVC1G04DBVR, U46 SN74LVC1G08DBVR, U47 SN74LVC1G08DBVR, U48 SN74LVC1G08DBVR, U49 SN74LVC1G08DBVR, U5 TPS25200DRVR, U50 SN74LVC1G08DBVR, U51 SN74LVC1G08DBVR, U52 SN74LVC1G08DBVR, U53 SN74LVC1G08DBVR, U54 TPS3808G33DBVR, U55 TLV3011BIDBVR, U56 SN74LVC1G08DBVR, U6 TPS63070RNMR, U60 CAT4101TV-T75, U61 CAT4101TV-T75, U62 SN74LVC1G125DBVR, U63 SN74LVC1G125DBVR, U7 TP4056-42-ESOP8, U70 MP3435GL-Z, U8 TLV3011BIDBVR, U9 TPS3808G33DBVR

Commit message: Update title blocks to Rev A prototype candidate, add comprehensive design review, and enhance README
Other:
- company: (none) -> Hector Jimenez
- title: ROUND LED FLASH - ENGINEERING DRAFT -> Round LED Flash — Annular Ring Camera Strobe
Changed lines of the file:
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@@
 (kicad_sch (version 20250114) (generator "eeschema") (generator_version "10.0")
  (paper "User" 1189 1189)
-(title_block (title "ROUND LED FLASH - ENGINEERING DRAFT") (date "2026-10-20") (rev "A-draft") (comment 1 "Incomplete electrical design - NOT FOR FABRICATION"))
+(title_block (title "Round LED Flash — Annular Ring Camera Strobe") (date "2026-10-21") (rev "Rev A") (company "Hector Jimenez") (comment 1 "Engineering prototype candidate — bench qualification pending"))
 (wire (pts (xy 49.5300 55.8800) (xy 46.9900 55.8800)) (stroke (width 0) (type default)))
 (label "BAT_PROT" (at 46.9900 55.8800 180) (effects (font (size 0.9 0.9)) (justify left bottom)))
